Commit message: Deleted spaces. Shift manipulator base frame and add camera frame.

File: robots/youbot.urdf.xacro (robot description, xacro)
@@ -12,8 +12,12 @@
   <!-- youbot plate -->
   <xacro:include filename="$(find youbot_description)/urdf/youbot_plate/plate.urdf.xacro" />
+  <!-- manipulator plate -->
+  <xacro:include filename="$(find youbot_description)/urdf/manipulator_plate/manipulator_plate.urdf.xacro" />
   <!-- youbot arm -->
   <xacro:include filename="$(find youbot_description)/urdf/youbot_arm/arm.urdf.xacro"/>
   <!-- youbot gripper -->
   <xacro:include filename="$(find youbot_description)/urdf/youbot_gripper/gripper.urdf.xacro" />
+  <!-- camera -->
+  <xacro:include filename="$(find youbot_description)/urdf/sensors/realsense_sr300.urdf.xacro" />
   <!-- controller manager -->
   <xacro:include filename="$(find youbot_description)/controller/ros_controller.urdf.xacro" />
@@ -35,10 +39,16 @@
     <origin xyz="-0.159 0 0.046" rpy="0 0 0" />
   </xacro:youbot_plate>
-  <xacro:youbot_arm name="arm" parent="base_link">
-    <origin xyz="0.143 0 0.046" rpy="0 0 0" />
+  <xacro:manipulator_plate name="m_plate" parent="base_link">
+    <origin xyz="0.166 0 0.034" rpy="0 0 0" />                  <!-- 11+23 -->
+  </xacro:manipulator_plate>
+  <xacro:youbot_arm name="arm" parent="m_plate_link">
+    <origin xyz="0.098 0 0.035" rpy="0 0 0" />                  <!-- -23+121 -->
   </xacro:youbot_arm>
   <xacro:youbot_gripper name="gripper" parent="arm_link_5">
     <origin xyz="0 0 0" rpy="0 0 0" />
   </xacro:youbot_gripper>
+  <xacro:realsense_sr300_camera name="realsense" parent="arm_link_5">
+    <origin xyz="-0.05532 -0.0323613 0.0594661" rpy="0.0462514 -0.00565613 1.55401" />
+  </xacro:realsense_sr300_camera>
   <!-- base laser front -->
   <xacro:hokuyo_urg04_laser name="base_laser_front" parent="base" ros_topic="base_scan" update_rate="10" min_angle="-1.57" max_angle="1.57">

File: urdf/youbot_arm/arm.urdf.xacro (robot description, xacro)
@@ -189,5 +189,5 @@
 			<dynamics damping="1" friction="1" />
 			<limit effort="1" velocity="${M_PI / 2.0}" lower="0" upper="${joint_5_limit}" />
-                        <safety_controller k_position="20" k_velocity="100" soft_lower_limit="0" soft_upper_limit="${joint_5_limit_soft}" />
+			<safety_controller k_position="20" k_velocity="100" soft_lower_limit="0" soft_upper_limit="${joint_5_limit_soft}" />
 		</joint>
 		<link name="${name}_link_5">

Commit message: Rename camera topic

File: robots/youbot.urdf.xacro (robot description, xacro)
@@ -48,5 +48,5 @@
     <origin xyz="0 0 0" rpy="0 0 0" />
   </xacro:youbot_gripper>
-  <xacro:realsense_sr300_camera name="realsense" parent="arm_link_5">
+  <xacro:realsense_sr300_camera name="camera_ir_optical_frame" parent="arm_link_5">
     <origin xyz="-0.05532 -0.0323613 0.0594661" rpy="0.0462514 -0.00565613 1.55401" />
   </xacro:realsense_sr300_camera>

File: urdf/sensors/realsense_sr300.urdf.xacro (robot description, xacro)
@@ -8,7 +8,7 @@
 		<xacro:insert_block name="origin" />
 		<parent link="${parent}" />
-		<child link="${name}_camera_ir" />
+		<child link="${name}" />
 	</joint>
-	<link name="${name}_camera_ir">
+	<link name="${name}">
 <!--       <visual>
         <origin xyz="0 0 0" rpy="0 0 0" />

Commit message: Change camera frame rotation

File: robots/youbot.urdf.xacro (robot description, xacro)
@@ -49,5 +49,5 @@
   </xacro:youbot_gripper>
   <xacro:realsense_sr300_camera name="realsense_camera" parent="arm_link_5">
-    <origin xyz="-0.05532 -0.0323613 0.0594661" rpy="0.0462514 -0.00565613 1.55401" />
+    <origin xyz="-0.05532 -0.0323613 0.0594661" rpy="-0.0064 -0.0461 -1.5540" />
   </xacro:realsense_sr300_camera>
   <!-- base laser front -->
